File: STM32G0XJX-breakout.kicad_sch (KiCad schematic)
At the start: 5 parts, among them J1 PinHeader 1x4 2.54mm, J2 PinHeader 1x4 2.54mm, U1 STM32C011J6Mx

Commit message: done
Parts:
- removed U1: STM32C011J6Mx, Package_SO:SOIC-8_3.9x4.9mm_P1.27mm, symbol MCU_ST_STM32C0:STM32C011J6Mx
- added U2: STM32G031J6Mx, Package_SO:JEITA_SOIC-8_3.9x4.9mm_P1.27mm, symbol MCU_ST_STM32G0:STM32G031J6Mx
- C1: value 100n -> 2u2; footprint Capacitor_SMD:C_0805_2012Metric -> Capacitor_SMD:C_0603_1608Metric
- C2: value 4u7 -> 2u2; footprint Capacitor_SMD:C_0805_2012Metric -> Capacitor_SMD:C_0603_1608Metric
Connections:
- net +3.3V: now also U2.2 (VDD)
- net GND: now also U2.3 (VSS)
- net PA0/PA1/PA2/PF2: now also U2.4 (PA0/PA1/PA2/PF2)
- net PA10/PA12: now also U2.6 (PA10/PA12)
- net PA13: now also U2.7 (PA13)
- net PA14/PB6/PC15 renamed PA14/PA15/PB5/PB6
- net PA14/PA15/PB5/PB6: now also U2.8 (PA14/PA15/PB5/PB6)
- net PA8/PA9/PA11 renamed PA8/PA9/PA11/PB0/PB1
- net PA8/PA9/PA11/PB0/PB1: now also U2.5 (PA8/PA9/PA11/PB0/PB1)
- net PB7/PC14 renamed PB7/PB8/PB9/PC14
- net PB7/PB8/PB9/PC14: now also U2.1 (PB7/PB8/PB9/PC14)
Changed lines of the file:
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@@
 	(wire
 		(pts
-			(xy 189.23 101.6) (xy 170.18 101.6)
+			(xy 175.26 104.14) (xy 200.66 104.14)
 		)
 		(stroke
@@
 	(wire
 		(pts
-			(xy 257.81 48.26) (xy 240.03 48.26)
+			(xy 265.43 48.26) (xy 240.03 48.26)
 		)
 		(stroke
@@
 	(wire
 		(pts
-			(xy 189.23 109.22) (xy 170.18 109.22)
-		)
-		(stroke
-			(width 0)
-			(type default)
-		)
-	)
-	(wire
-		(pts
-			(xy 107.95 101.6) (xy 119.38 101.6)
-		)
-		(stroke
-			(width 0)
-			(type default)
-		)
-	)
-	(wire
-		(pts
-			(xy 189.23 104.14) (xy 170.18 104.14)
+			(xy 175.26 106.68) (xy 200.66 106.68)
+		)
+		(stroke
+			(width 0)
+			(type default)
+		)
+	)
+	(wire
+		(pts
+			(xy 92.71 101.6) (xy 114.3 101.6)
+		)
+		(stroke
+			(width 0)
+			(type default)
+		)
+	)
+	(wire
+		(pts
+			(xy 175.26 109.22) (xy 200.66 109.22)
+		)
+		(stroke
+			(width 0)
+			(type default)
+		)
+	)
+	(wire
+		(pts
+			(xy 175.26 101.6) (xy 200.66 101.6)
 		)
 		(stroke
@@
 	(wire
 		(pts
-			(xy 189.23 111.76) (xy 170.18 111.76)
-		)
-		(stroke
-			(width 0)
-			(type default)
-		)
-	)
-	(wire
-		(pts
 			(xy 144.78 119.38) (xy 144.78 121.92)
 		)
@@
 	(wire
 		(pts
-			(xy 257.81 55.88) (xy 240.03 55.88)
-		)
-		(stroke
-			(width 0)
-			(type default)
-		)
-	)
-	(wire
-		(pts
-			(xy 257.81 53.34) (xy 240.03 53.34)
+			(xy 265.43 55.88) (xy 240.03 55.88)
+		)
+		(stroke
+			(width 0)
+			(type default)
+		)
+	)
+	(wire
+		(pts
+			(xy 265.43 53.34) (xy 240.03 53.34)
 		)
 		(stroke
@@
 	(wire
 		(pts
-			(xy 257.81 50.8) (xy 240.03 50.8)
+			(xy 265.43 50.8) (xy 240.03 50.8)
 		)
 		(stroke
@@
 	(wire
 		(pts
-			(xy 189.23 106.68) (xy 170.18 106.68)
-		)
-		(stroke
-			(width 0)
-			(type default)
-		)
-	)
-	(label "PA13"
-		(at 257.81 50.8 180)
-		(effects
-			(font
-				(size 1.27 1.27)
-			)
-			(justify right bottom)
-		)
-	)
-	(label "PA10{slash}PA12"
-		(at 189.23 106.68 180)
-		(effects
-			(font
-				(size 1.27 1.27)
-			)
-			(justify right bottom)
-		)
-	)
-	(label "PA14{slash}PB6{slash}PC15"
-		(at 189.23 111.76 180)
-		(effects
-			(font
-				(size 1.27 1.27)
-			)
-			(justify right bottom)
-		)
-	)
-	(label "PA10{slash}PA12"
-		(at 257.81 53.34 180)
-		(effects
-			(font
-				(size 1.27 1.27)
-			)
-			(justify right bottom)
-		)
-	)
-	(label "PA8{slash}PA9{slash}PA11"
-		(at 189.23 104.14 180)
-		(effects
-			(font
-				(size 1.27 1.27)
-			)
-			(justify right bottom)
-		)
-	)
-	(label "PA0{slash}PA1{slash}PA2{slash}PF2"
-		(at 189.23 101.6 180)
-		(effects
-			(font
-				(size 1.27 1.27)
-			)
-			(justify right bottom)
-		)
-	)
-	(label "PB7{slash}PC14"
-		(at 180.34 48.26 0)
-		(effects
-			(font
-				(size 1.27 1.27)
-			)
-			(justify left bottom)
-		)
-	)
-	(label "PA8{slash}PA9{slash}PA11"
-		(at 257.81 55.88 180)
-		(effects
-			(font
-				(size 1.27 1.27)
-			)
-			(justify right bottom)
+			(xy 175.26 111.76) (xy 200.66 111.76)
+		)
+		(stroke
+			(width 0)
+			(type default)
 		)
 	)
@@
 		)
 	)
-	(label "PB7{slash}PC14"
-		(at 107.95 101.6 0)
+	(label "PA10{slash}PA12"
+		(at 200.66 106.68 180)
 		(effects
 			(font
 				(size 1.27 1.27)
 			)
-			(justify left bottom)
-		)
-	)
-	(label "PA13"
-		(at 189.23 109.22 180)
+			(justify right bottom)
+		)
+	)
+	(label "PA14{slash}PA15{slash}PB5{slash}PB6"
+		(at 200.66 111.76 180)
 		(effects
 			(font
@@
 		)
 	)
-	(label "PA14{slash}PB6{slash}PC15"
-		(at 257.81 48.26 180)
+	(label "PA8{slash}PA9{slash}PA11{slash}PB0{slash}PB1"
+		(at 200.66 104.14 180)
+		(effects
+			(font
+				(size 1.27 1.27)
+			)
+			(justify right bottom)
+		)
+	)
+	(label "PA14{slash}PA15{slash}PB5{slash}PB6"
+		(at 265.43 48.26 180)
+		(effects
+			(font
+				(size 1.27 1.27)
+			)
+			(justify right bottom)
+		)
+	)
+	(label "PA0{slash}PA1{slash}PA2{slash}PF2"
+		(at 200.66 101.6 180)
+		(effects
+			(font
+				(size 1.27 1.27)
+			)
+			(justify right bottom)
+		)
+	)
+	(label "PA8{slash}PA9{slash}PA11{slash}PB0{slash}PB1"
+		(at 265.43 55.88 180)
+		(effects
+			(font
+				(size 1.27 1.27)
+			)
+			(justify right bottom)
+		)
+	)
+	(label "PA13"
+		(at 265.43 50.8 180)
+		(effects
+			(font
+				(size 1.27 1.27)
+			)
+			(justify right bottom)
+		)
+	)
+	(label "PB7{slash}PB8{slash}PB9{slash}PC14"
+		(at 180.34 48.26 0)
+		(effects
+			(font
+				(size 1.27 1.27)
+			)
+			(justify left bottom)
+		)
+	)
+	(label "PB7{slash}PB8{slash}PB9{slash}PC14"
+		(at 92.71 101.6 0)
+		(effects
+			(font
+				(size 1.27 1.27)
+			)
+			(justify left bottom)
+		)
+	)
+	(label "PA13"
+		(at 200.66 109.22 180)
+		(effects
+			(font
+				(size 1.27 1.27)
+			)
+			(justify right bottom)
+		)
+	)
+	(label "PA10{slash}PA12"
+		(at 265.43 53.34 180)
 		(effects
 			(font
@@
 			)
 		)
-		(property "Value" "4u7"
+		(property "Value" "2u2"
 			(at 171.45 67.31 0)
 			(show_name no)
@@
 			)
 		)
-		(property "Footprint" "Capacitor_SMD:C_0805_2012Metric"
+		(property "Footprint" "Capacitor_SMD:C_0603_1608Metric"
 			(at 171.1452 68.58 0)
 			(hide yes)
@@
 			)
 		)
-		(property "Value" "100n"
+		(property "Value" "2u2"
 			(at 161.29 67.31 0)
 			(show_name no)
@@
 			)
 		)
-		(property "Footprint" "Capacitor_SMD:C_0805_2012Metric"
+		(property "Footprint" "Capacitor_SMD:C_0603_1608Metric"
 			(at 160.9852 68.58 0)
 			(hide yes)
@@
 	)
 	(symbol
-		(lib_id "MCU_ST_STM32C0:STM32C011J6Mx")
+		(lib_id "MCU_ST_STM32G0:STM32G031J6Mx")
 		(at 144.78 106.68 0)
 		(unit 1)
@@
 		(in_pos_files yes)
 		(dnp no)
-		(fields_autoplaced yes)
-		(property "Reference" "U1"
-			(at 146.9233 91.44 0)
+		(property "Reference" "U2"
+			(at 118.11 95.25 0)
 			(show_name no)
 			(do_not_autoplace no)
@@
 			)
 		)
-		(property "Value" "STM32C011J6Mx"
-			(at 146.9233 93.98 0)
+		(property "Value" "STM32G031J6Mx"
+			(at 118.11 118.11 0)
 			(show_name no)
 			(do_not_autoplace no)
@@
 			)
 		)
-		(property "Footprint" "Package_SO:SOIC-8_3.9x4.9mm_P1.27mm"
-			(at 121.92 116.84 0)
+		(property "Footprint" "Package_SO:JEITA_SOIC-8_3.9x4.9mm_P1.27mm"
+			(at 116.84 116.84 0)
 			(hide yes)
 			(show_name no)
@@
 			)
 		)
-		(property "Datasheet" "https://www.st.com/resource/en/datasheet/stm32c011j6.pdf"
+		(property "Datasheet" "https://www.st.com/resource/en/datasheet/stm32g031j6.pdf"
 			(at 144.78 106.68 0)
 			(hide yes)
@@
 			)
 		)
-		(property "Description" "STMicroelectronics Arm Cortex-M0+ MCU, 32KB flash, 6KB RAM, 48 MHz, 2.0-3.6V, 6 GPIO, SO8N"
+		(property "Description" "STMicroelectronics Arm Cortex-M0+ MCU, 32KB flash, 8KB RAM, 64 MHz, 1.7-3.6V, 6 GPIO, SO8N"
 			(at 144.78 106.68 0)
 			(hide yes)
@@
 			)
 		)
+		(pin "1"
+		)
 		(pin "8"
 		)
+		(pin "3"
+		)
+		(pin "5"
+		)
+		(pin "4"
+		)
+		(pin "2"
+		)
+		(pin "6"
+		)
 		(pin "7"
-		)
-		(pin "6"
-		)
-		(pin "5"
-		)
-		(pin "4"
-		)
-		(pin "3"
-		)
-		(pin "2"
-		)
-		(pin "1"
 		)
 		(instances
 			(project "STM32G0XJX-breakout"
 				(path "/ddb69247-eed9-4f3f-9fd5-97496ec47cb8"
-					(reference "U1")
+					(reference "U2")
 					(unit 1)
 				)
